File: Rev1/PowerShield.brd (EAGLE design)
At the start: 42.2 x 23.1 mm, 39 parts, among them U1 MCP73831

Commit message: Add Rev2 files
Parts:
- added CN1: (no value), adafruit:JST-PH-2-THM-RA
- added R5: 1M, LowPowerLab:0603-RES
- added R6: 180K, LowPowerLab:0603-RES
- added R7: 110K, LowPowerLab:0603-RES
- added U$26: JUMPER_3, LowPowerLab:JUMPER_3
- C1: value 1u -> 10u; device LowPowerLab:0603-CAP -> LowPowerLab:0805-CAP-LARGEPADS
- L1: value 10uH -> 4.7uH
- U$2: value LT3525 -> TPS61222SOT363
- moved C1 6.90 mm to (28.6, 17.7), turned to 270 degrees
- moved C2 3.87 mm to (18.0, 17.9), turned to 90 degrees
- moved U$3 1.65 mm to (5.46, 17.0)
- moved L1 1.17 mm to (31.4, 17.5)
- moved CN3 1.02 mm to (5.97, 5.84), turned to 90 degrees
- moved U$2 0.40 mm to (25.5, 17.7)
Connections:
- new net N$1: L1.P$1, U$2.5
- new net N$5: R7.2, U$26.1
- new net N$7: R5.1, U$2.2, U$26.2
- net GND: now also CN1.2, R6.1, R7.1, U$2.3; no longer U$13.1, U$13.2, U$17.1, U$17.2, U$2.2, U$2.5, U$21.1, U$21.2, U$23.1, U$23.2, U$9.1, U$9.2
- net N$4: now also R6.2, U$26.3; no longer L1.P$1, U$2.6
- net VBAT: now also CN1.1
- net VBAT_SWITCHED: now also U$2.6; no longer U$2.3
- net VIN_MOTEINO: now also R5.2
Routing:
- net GND: track 44.3 -> 20.4 mm, vias 9 -> 8
- net N$60: track 10.2 -> 0.00 mm
- net VBAT: track 51.5 -> 43.4 mm
- net N$7: track 0.00 -> 6.93 mm, vias 0 -> 1
- net N$1: track 0.00 -> 5.54 mm, vias 1 -> 0
- net N$9: track 5.08 -> 0.00 mm
- net N$8: track 5.08 -> 0.00 mm
- net N$13: track 5.08 -> 0.00 mm
- net N$12: track 5.08 -> 0.00 mm
- net N$11: track 5.08 -> 0.00 mm
- net N$10: track 5.08 -> 0.00 mm
- net VBAT_SWITCHED: track 28.5 -> 23.5 mm
- net N$4: track 4.16 -> 1.49 mm, vias 0 -> 1
- net N$5: track 0.00 -> 2.44 mm, vias 0 -> 1
Other:
- outline, holes or cut-outs redrawn
- board text added: "(5V)"
- board text added: "1-14-2014"
- board text added: "3.3V"
- board text added: "LowPowerLab"
- board text added: "OUTPUT"
- board text added: "R1"
- board text added: "VBAT"
- board text added: "or AA/AAA"
- board text removed: "+"
- board text removed: "-"
- board text removed: "5-14-2014"
- board text removed: "AA/AAA"
- board text removed: "Charging"
- board text removed: "LowPowerLab.com"
- board text removed: "Rev2"
- board text removed: "USB for Lipo charging ONLY!"
- board text removed: "VIN"
- board text removed: "VOUT"
- board text removed: "or"
