File: Rev1/PowerShield.sch (EAGLE design)
At the start: 38 parts, among them U1 MCP73831

Commit message: Add Rev2 files
Parts:
- added CN1: (no value), adafruit:JST_2PIN-THM-RA
- added R5: 1M, LowPowerLab:RESISTOR0603-RES
- added R6: 180K, LowPowerLab:RESISTOR0603-RES
- added R7: 110K, LowPowerLab:RESISTOR0603-RES
- added U$26: JUMPER_3, LowPowerLab:JUMPER_3
- C1: value 1u -> 10u; device LowPowerLab:CAP0603-CAP -> LowPowerLab:CAP0805-CAP-LARGEPADS
- L1: value 10uH -> 4.7uH
- U$2: value LT3525 -> TPS61222SOT363; device LowPowerLab:LT3525 -> LowPowerLab:TPS61222SOT363
Connections:
- new net N$1: L1.1, U$2.L
- new net N$5: R7.2, U$26.P$1
- new net N$7: R5.1, U$2.FB, U$26.P$2
- net GND: now also CN1.1, R6.1, R7.1, U$2.GND; no longer U$13.P$1, U$13.P$2, U$17.P$1, U$17.P$2, U$2.GND1, U$2.GND2, U$21.P$1, U$21.P$2, U$23.P$1, U$23.P$2, U$9.P$1, U$9.P$2
- net N$4: now also R6.2, U$26.P$3; no longer L1.1, U$2.SW
- net VBAT: now also CN1.2
- net VBAT_SWITCHED: now also U$2.EN; no longer U$2.SHDN
- net VIN_MOTEINO: now also R5.2
Other:
- note added: "PowerShield R1"
- note added: "TPS61220"
- note added: "http://lowpowerlab.com"
- note removed: "PowerShield R2"
- note removed: "http://lowpowerlab.com/powershield"
- moved on the sheet: C1, C2, L1
